File: System 100 PS22-PS24.sch (KiCad schematic (older format))
At the start: 40 parts, among them P1 CONN_01X01, P10 CONN_01X01, P11 CONN_01X01, P12 CONN_01X01, P13 CONN_01X01, P2 CONN_01X01, P3 CONN_01X01, P4 CONN_01X01, Q101 TIP31A, Q102 TIP31A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

Commit message: footprints assigned
Parts:
- removed P12: CONN_01X01, symbol CONN_01X01
- C101, C102: footprint (none) -> MyModules:5MM-POL-CAP
- C103, C104: footprint (none) -> Capacitors_THT:C_Disc_D6_P5
- C105, C106: footprint (none) -> MyModules:2MM-POL-CAP
- D101, D101-1, D102, D102-1, D103, D103-1, D104, D104-1, D105, D106: footprint (none) -> Diodes_THT:Diode_DO-41_SOD81_Horizontal_RM10
- F101, F102: footprint (none) -> Fuse_Holders_and_Fuses:Fuseholder5x20_horiz_open_inline_Type-I
- P10, P13: value CONN_01X01 -> CONN_01X04; symbol CONN_01X01 -> CONN_01X04
- P11: value CONN_01X01 -> CONN_01X06; symbol CONN_01X01 -> CONN_01X06
- P5: renamed from P?; footprint (none) -> w_conn_kk156:kk156_26-60-4080
- Q101, Q102: footprint (none) -> TO_SOT_Packages_THT:TO-220_Neutral123_Horizontal_LargePads
- R101, R102, R104, R105, R107: footprint (none) -> Resistors_THT:Resistor_Horizontal_RM10mm
- R103: renamed from 3.3K; value R103 -> 3.3K; footprint (none) -> Resistors_THT:Resistor_Horizontal_RM10mm
- R106: renamed from 3.3K?; value R106 -> 3.3K; footprint (none) -> Resistors_THT:Resistor_Horizontal_RM10mm
- U101, U102: footprint (none) -> Housings_DIP:DIP-14_W7.62mm
- VR101, VR102: footprint (none) -> MyModules:Bourns_3362P
Connections:
- net GND: now also P11.2 (P2), P11.3 (P3), P11.4 (P4), P11.5 (P5), P11.6 (P6); no longer U102.3 (CS)
- net at C105.1 (+), D105.1 (K), P10.1 (P1)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: now also P10.2 (P2), P10.3 (P3), P10.4 (P4)
- net at C102.2 (-), C106.2 (-), D103-1.2 (A)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: now also P13.2 (P2), P13.3 (P3), P13.4 (P4)

Commit message: routed
Parts:
- P1, P2, P3, P4: footprint (none) -> Pin_Headers:Pin_Header_Straight_1x01
- P10, P13: footprint (none) -> Pin_Headers:Pin_Header_Straight_1x04
- P11: footprint (none) -> Pin_Headers:Pin_Header_Straight_2x03
Connections:
- net GND: now also U102.3 (CS)
Changed lines of the file:
@@
 F 0 "P2" H 3100 6825 50  0000 C CNN
 F 1 "CONN_01X01" V 3200 6725 50  0000 C CNN
-F 2 "" H 3100 6725 60  0001 C CNN
+F 2 "Pin_Headers:Pin_Header_Straight_1x01" H 3100 6725 60  0001 C CNN
 F 3 "" H 3100 6725 60  0000 C CNN
 	1    3100 6725
@@
 F 0 "P3" H 2500 6825 50  0000 C CNN
 F 1 "CONN_01X01" V 2600 6725 50  0000 C CNN
-F 2 "" H 2500 6725 60  0001 C CNN
+F 2 "Pin_Headers:Pin_Header_Straight_1x01" H 2500 6725 60  0001 C CNN
 F 3 "" H 2500 6725 60  0000 C CNN
 	1    2500 6725
@@
 F 0 "P10" H 2675 425 50  0000 C CNN
 F 1 "CONN_01X04" V 2775 750 50  0000 C CNN
-F 2 "" H 2675 750 60  0001 C CNN
+F 2 "Pin_Headers:Pin_Header_Straight_1x04" H 2675 750 60  0001 C CNN
 F 3 "" H 2675 750 60  0000 C CNN
 	1    2675 750
@@
 F 0 "P11" H 4550 425 50  0000 C CNN
 F 1 "CONN_01X06" V 4650 775 50  0000 C CNN
-F 2 "" H 4550 775 60  0001 C CNN
+F 2 "Pin_Headers:Pin_Header_Straight_2x03" H 4550 775 60  0001 C CNN
 F 3 "" H 4550 775 60  0000 C CNN
 	1    4550 775
@@
 F 0 "P1" H 6450 6825 50  0000 C CNN
 F 1 "CONN_01X01" V 6550 6725 50  0000 C CNN
-F 2 "" H 6450 6725 60  0001 C CNN
+F 2 "Pin_Headers:Pin_Header_Straight_1x01" H 6450 6725 60  0001 C CNN
 F 3 "" H 6450 6725 60  0000 C CNN
 	1    6450 6725
@@
 F 0 "P4" H 5850 6825 50  0000 C CNN
 F 1 "CONN_01X01" V 5950 6725 50  0000 C CNN
-F 2 "" H 5850 6725 60  0001 C CNN
+F 2 "Pin_Headers:Pin_Header_Straight_1x01" H 5850 6725 60  0001 C CNN
 F 3 "" H 5850 6725 60  0000 C CNN
 	1    5850 6725
@@
 F 0 "P13" H 7500 1000 50  0000 C CNN
 F 1 "CONN_01X04" V 7600 750 50  0000 C CNN
-F 2 "" H 7500 750 60  0001 C CNN
+F 2 "Pin_Headers:Pin_Header_Straight_1x04" H 7500 750 60  0001 C CNN
 F 3 "" H 7500 750 60  0000 C CNN
 	1    7500 750
@@
 Wire Wire Line
 	6175 1150 6175 2025
+Wire Wire Line
+	8025 1250 6175 1250
+Wire Wire Line
+	6175 1250 6175 2725
 $EndSCHEMATC

Commit message: gerbers generated, ready to order
Other:
- note added: "0.5A FUSE for PS24 (220V)\nJUMPER for PS22 (110V)"
- note added: "BLK"
- note added: "GRY"
- note added: "RED"
- note added: "YEL"
Changed lines of the file:
@@
 LIBS:valves
 LIBS:MySynthParts
+LIBS:System 100 PS22-PS24-cache
 EELAYER 25 0
 EELAYER END
@@
 Connection ~ 7350 1150
 Wire Wire Line
-	6175 1150 6175 2025
-Wire Wire Line
-	8025 1250 6175 1250
-Wire Wire Line
-	6175 1250 6175 2725
+	6175 1150 6175 2725
+Text Notes 3200 6175 0    50   ~ 0
+0.5A FUSE for PS24 (220V)\nJUMPER for PS22 (110V)
+Text Notes 6550 6150 0    50   ~ 0
+0.5A FUSE for PS24 (220V)\nJUMPER for PS22 (110V)
+Text Notes 2400 6975 0    80   ~ 0
+YEL
+Text Notes 2975 6975 0    80   ~ 0
+GRY
+Text Notes 5725 6975 0    80   ~ 0
+RED
+Text Notes 6325 6975 0    80   ~ 0
+BLK
 $EndSCHEMATC
