File: System 100 PS22-PS24.kicad_pcb (KiCad board)
At the start: 2 copper layers, 43 parts, among them P1 CONN_01X01, P10 CONN_01X04, P11 CONN_01X06, P13 CONN_01X04, P2 CONN_01X01, P3 CONN_01X01, P4 CONN_01X01, P5 CONN_01X08, Q101 TIP31A, Q102 TIP31A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

Commit message: gerbers generated, ready to order
Parts:
- F101, F102: value PS24:FUSE -> PS24: 0.5A
Routing:
- net GND: track 0.00 -> 3.49 mm
- net Net-(Q101-Pad3): track 32.8 -> 35.3 mm
- net Net-(C103-Pad2): track 11.4 -> 13.2 mm
- net Net-(Q102-Pad3): track 34.9 -> 35.9 mm
Other:
- board text added: "Roland"
Changed lines of the file:
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@@
     (area 61.841667 37.899999 193.100001 138.100001)
     (thickness 1.6)
-    (drawings 31)
-    (tracks 196)
+    (drawings 46)
+    (tracks 205)
     (zones 0)
     (modules 43)
@@
     (40 Dwgs.User user)
     (41 Cmts.User user)
-    (42 Eco1.User user hide)
+    (42 Eco1.User user)
     (43 Eco2.User user)
     (44 Edge.Cuts user)
@@
   )
   (setup
-    (last_trace_width 1)
+    (last_trace_width 0.5)
     (user_trace_width 0.25)
     (user_trace_width 0.5)
@@
     (mod_text_size 1 1)
     (mod_text_width 0.15)
-    (pad_size 52 20)
+    (pad_size 50 20)
     (pad_drill 0)
     (pad_to_mask_clearance 0.2)
@@
     (visible_elements 7FFEF7FF)
     (pcbplotparams
-      (layerselection 0x00030_80000001)
-      (usegerberextensions false)
+      (layerselection 0x010f0_80000001)
+      (usegerberextensions true)
       (excludeedgelayer true)
       (linewidth 0.200000)
@@
       (psa4output false)
       (plotreference true)
-      (plotvalue true)
+      (plotvalue false)
       (plotinvisibletext false)
       (padsonsilk false)
-      (subtractmaskfromsilk false)
+      (subtractmaskfromsilk true)
       (outputformat 1)
       (mirror false)
-      (drillshape 1)
+      (drillshape 0)
       (scaleselection 1)
-      (outputdirectory ""))
+      (outputdirectory Gerbers/))
   )
   (net 0 "")
@@
       (net 23 "Net-(Q101-Pad3)"))
     (pad "" thru_hole circle (at 0 -16.764 90) (size 4 4) (drill 3.79984) (layers *.Cu *.Mask F.SilkS))
-    (pad "" smd rect (at 0 -13.5) (size 38 20) (layers F.Cu F.Paste F.Mask))
-    (pad 0 smd rect (at 6 -13.5) (size 50 20) (layers B.Cu F.Paste F.Mask))
+    (pad "" smd rect (at 6 -13.5) (size 50 20) (layers F.Cu F.Paste F.Mask))
+    (pad 0 smd rect (at 6 -13.5) (size 50 20) (layers B.Cu F.Paste B.Mask))
     (pad "" thru_hole circle (at -17 -22) (size 1.524 1.524) (drill 0.5) (layers *.Cu *.Mask F.SilkS))
     (pad "" thru_hole circle (at -14 -22) (size 1.524 1.524) (drill 0.5) (layers *.Cu *.Mask F.SilkS))
@@
       (net 25 "Net-(Q102-Pad3)"))
     (pad "" thru_hole circle (at 0 -16.764 270) (size 4 4) (drill 3.79984) (layers *.Cu *.Mask F.SilkS))
-    (pad "" smd rect (at 0 -13.5 180) (size 38 20) (layers F.Cu F.Paste F.Mask))
-    (pad 0 smd rect (at -6 -13.5 180) (size 52 20) (layers B.Cu F.Paste F.Mask))
+    (pad "" smd rect (at -6 -13.5 180) (size 50 20) (layers F.Cu F.Paste F.Mask))
+    (pad 0 smd rect (at -6 -13.5 180) (size 50 20) (layers B.Cu F.Paste B.Mask))
     (pad "" thru_hole circle (at -17 -22 180) (size 1.524 1.524) (drill 0.5) (layers *.Cu *.Mask F.SilkS))
     (pad "" thru_hole circle (at -14 -22 180) (size 1.524 1.524) (drill 0.5) (layers *.Cu *.Mask F.SilkS))
@@
       (effects (font (thickness 0.3048)))
     )
-    (fp_text value PS24:FUSE (at -3.5 -19 360) (layer F.SilkS)
+    (fp_text value "PS24: 0.5A" (at -5 -15 450) (layer F.SilkS)
       (effects (font (thickness 0.3048)))
     )
@@
       (effects (font (thickness 0.3048)))
     )
-    (fp_text value PS24:FUSE (at -3.5 -19 360) (layer F.SilkS)
+    (fp_text value "PS24: 0.5A" (at -0.1 -19.4 360) (layer F.SilkS) hide
       (effects (font (thickness 0.3048)))
     )
@@
     (pad 1 thru_hole rect (at 0 0) (size 2.5 2.5) (drill 1.2) (layers *.Cu *.Mask)
       (net 17 "Net-(P4-Pad1)"))
+  )
+  (gr_circle (center 178 123) (end 179.5 123.75) (layer Eco1.User) (width 0.2))
+  (gr_circle (center 178 53) (end 179.25 54) (layer Eco1.User) (width 0.2))
+  (gr_circle (center 78 53) (end 79.25 54) (layer Eco1.User) (width 0.2))
+  (gr_circle (center 78 123) (end 79 124.25) (layer Eco1.User) (width 0.2))
+  (gr_line (start 78 123) (end 78 126.25) (angle 90) (layer Eco1.User) (width 0.2))
+  (gr_line (start 78 123) (end 74.75 123) (angle 90) (layer Eco1.User) (width 0.2))
+  (gr_line (start 178 53) (end 181.25 53) (angle 90) (layer Eco1.User) (width 0.2))
+  (gr_line (start 178 53) (end 178 49.75) (angle 90) (layer Eco1.User) (width 0.2))
+  (gr_line (start 178 123) (end 181.25 123) (angle 90) (layer Eco1.User) (width 0.2))
+  (gr_line (start 178 123) (end 178 126.25) (angle 90) (layer Eco1.User) (width 0.2))
+  (gr_line (start 78 53) (end 78 49.75) (angle 90) (layer Eco1.User) (width 0.2))
+  (gr_line (start 78 53) (end 74.75 53) (angle 90) (layer Eco1.User) (width 0.2))
+  (gr_text Roland (at 69.25 132) (layer F.SilkS)
+    (effects (font (size 2 2) (thickness 0.3)))
+  )
+  (gr_text + (at 173 97.5) (layer F.SilkS)
+    (effects (font (size 2 2) (thickness 0.3)))
+  )
+  (gr_text + (at 173 82.25) (layer F.SilkS)
+    (effects (font (size 2 2) (thickness 0.3)))
   )
   (gr_text "PS22:\nJUMPER" (at 95 99) (layer F.SilkS)
@@
   (segment (start 97.00254 71) (end 97.00254 67.00508) (width 1) (layer B.Cu) (net 1) (status 10))
   (segment (start 97.00254 67.00508) (end 96.99746 67) (width 1) (layer B.Cu) (net 1) (status 30))
+  (segment (start 139.92 95.5) (end 139.92 94.36863) (width 0.5) (layer B.Cu) (net 2))
+  (segment (start 139.92 94.36863) (end 139.75 94.19863) (width 0.5) (layer B.Cu) (net 2))
+  (segment (start 140.28863 97) (end 140.75 97) (width 0.5) (layer B.Cu) (net 2))
+  (segment (start 139.92 95.5) (end 139.92 96.63137) (width 0.5) (layer B.Cu) (net 2))
+  (segment (start 139.92 96.63137) (end 140.28863 97) (width 0.5) (layer B.Cu) (net 2))
   (segment (start 108 118.5) (end 110.5 118.5) (width 1) (layer B.Cu) (net 3))
   (segment (start 121 106) (end 136 106) (width 1) (layer B.Cu) (net 3))
@@
   (segment (start 123 78.8) (end 123.8 78) (width 0.5) (layer B.Cu) (net 5))
   (segment (start 136.62 80.38) (end 136.62 81) (width 1) (layer F.Cu) (net 5))
-  (segment (start 123 75) (end 124.5 76.5) (width 0.5) (layer B.Cu) (net 6))
-  (segment (start 124.5 76.5) (end 130 76.5) (width 0.5) (layer B.Cu) (net 6))
-  (segment (start 130 76.5) (end 131.54 74.96) (width 0.5) (layer B.Cu) (net 6))
-  (segment (start 131.54 74.96) (end 131.54 73.38) (width 0.5) (layer B.Cu) (net 6))
+  (segment (start 124.75 71) (end 123 72.75) (width 0.5) (layer B.Cu) (net 6))
+  (segment (start 123 72.75) (end 123 75) (width 0.5) (layer B.Cu) (net 6))
+  (segment (start 130.29137 71) (end 124.75 71) (width 0.5) (layer B.Cu) (net 6))
+  (segment (start 131.54 73.38) (end 131.54 72.24863) (width 0.5) (layer B.Cu) (net 6))
+  (segment (start 131.54 72.24863) (end 130.29137 71) (width 0.5) (layer B.Cu) (net 6))
   (segment (start 137.38 95.5) (end 140.38 98.5) (width 0.5) (layer B.Cu) (net 7))
   (segment (start 148.75 103.25) (end 148.75 105.25) (width 0.5) (layer B.Cu) (net 7))
@@
   (segment (start 137.46 70.54863) (end 137.46 70.26) (width 1) (layer F.Cu) (net 22))
   (segment (start 137.46 67) (end 137.46 70.26) (width 1) (layer F.Cu) (net 22))
+  (segment (start 150 71.84) (end 150 74) (width 1) (layer F.Cu) (net 23))
+  (segment (start 150 74) (end 147.5 76.5) (width 1) (layer F.Cu) (net 23))
+  (segment (start 147.5 76.5) (end 134 76.5) (width 1) (layer F.Cu) (net 23))
+  (segment (start 134 76.5) (end 131.75 78.75) (width 1) (layer F.Cu) (net 23))
+  (segment (start 131.75 78.75) (end 131.75 80.79) (width 1) (layer F.Cu) (net 23))
+  (segment (start 131.75 80.79) (end 131.54 81) (width 1) (layer F.Cu) (net 23))
   (segment (start 150 71.84) (end 150 70) (width 1) (layer F.Cu) (net 23))
   (segment (start 150 70) (end 147 67) (width 1) (layer F.Cu) (net 23))
   (segment (start 147 67) (end 144.38963 67) (width 1) (layer F.Cu) (net 23))
   (segment (start 144.38963 67) (end 142.54 67) (width 1) (layer F.Cu) (net 23))
-  (segment (start 150 71.84) (end 145.34 76.5) (width 1) (layer F.Cu) (net 23))
-  (segment (start 132.339999 80.200001) (end 131.54 81) (width 1) (layer F.Cu) (net 23))
-  (segment (start 145.34 76.5) (end 136.04 76.5) (width 1) (layer F.Cu) (net 23))
-  (segment (start 136.04 76.5) (end 132.339999 80.200001) (width 1) (layer F.Cu) (net 23))
   (segment (start 136 105.5) (end 134.84 104.34) (width 1) (layer F.Cu) (net 24))
   (segment (start 134.84 104.34) (end 134.84 103.12) (width 1) (layer F.Cu) (net 24))
@@
   (segment (start 142.54 109) (end 142.54 106.24994) (width 1) (layer F.Cu) (net 24))
   (segment (start 142.54 106.24994) (end 141.79006 105.5) (width 1) (layer F.Cu) (net 24))
-  (segment (start 133.16 109) (end 135.61037 109) (width 1) (layer F.Cu) (net 25))
-  (segment (start 128.5 109) (end 133.16 109) (width 1) (layer F.Cu) (net 25))
-  (segment (start 126.5 107) (end 128.5 109) (width 1) (layer F.Cu) (net 25))
-  (segment (start 142.46 95.5) (end 138.96 99) (width 1) (layer F.Cu) (net 25))
-  (segment (start 138.96 99) (end 130.5 99) (width 1) (layer F.Cu) (net 25))
+  (segment (start 142.46 95.5) (end 142.46 97.29) (width 1) (layer F.Cu) (net 25))
+  (segment (start 142.46 97.29) (end 140.75 99) (width 1) (layer F.Cu) (net 25))
+  (segment (start 140.75 99) (end 130.5 99) (width 1) (layer F.Cu) (net 25))
   (segment (start 130.5 99) (end 126.5 103) (width 1) (layer F.Cu) (net 25))
   (segment (start 126.5 103) (end 126.5 107) (width 1) (layer F.Cu) (net 25))
+  (segment (start 126.5 107) (end 128.5 109) (width 1) (layer F.Cu) (net 25))
+  (segment (start 128.5 109) (end 133.16 109) (width 1) (layer F.Cu) (net 25))
+  (segment (start 133.16 109) (end 135.61037 109) (width 1) (layer F.Cu) (net 25))
   (segment (start 135.61037 109) (end 137.46 109) (width 1) (layer F.Cu) (net 25))
   (segment (start 169 74.54) (end 167.742765 74.54) (width 0.5) (layer B.Cu) (net 26))

Commit message: updated readme.md
Other:
- board outline added: 130 x 100 mm
Changed lines of the file:
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@@
   (page A4)
   (layers
-    (0 F.Cu signal)
-    (31 B.Cu signal)
+    (0 F.Cu signal hide)
+    (31 B.Cu signal hide)
     (32 B.Adhes user)
     (33 F.Adhes user)
@@
     (trace_min 0.2)
     (segment_width 0.2)
-    (edge_width 0.15)
+    (edge_width 0.2)
     (via_size 1)
     (via_drill 0.5)
@@
     (pad_to_mask_clearance 0.2)
     (aux_axis_origin 0 0)
-    (visible_elements 7FFEF7FF)
+    (visible_elements 7FFFF7FF)
     (pcbplotparams
       (layerselection 0x010f0_80000001)
@@
       (effects (font (size 1 1) (thickness 0.15)))
     )
-    (fp_text value 3.9 (at 5.08 3.81 90) (layer F.Fab)
+    (fp_text value 3.9 (at 5.2 0.075 90) (layer F.Fab)
       (effects (font (size 1 1) (thickness 0.15)))
     )
@@
       (effects (font (size 1 1) (thickness 0.15)))
     )
-    (fp_text value 3.3K (at 5.08 3.81 270) (layer F.Fab)
+    (fp_text value 3.3K (at 4.91 -0.225 270) (layer F.Fab)
       (effects (font (size 1 1) (thickness 0.15)))
     )
@@
       (effects (font (size 1 1) (thickness 0.15)))
     )
-    (fp_text value 3.3K (at 5.08 3.81) (layer F.Fab)
+    (fp_text value 3.3K (at 5.25 0.125) (layer F.Fab)
       (effects (font (size 1 1) (thickness 0.15)))
     )
@@
       (effects (font (size 1 1) (thickness 0.15)))
     )
-    (fp_text value 3.9 (at 5.08 3.81) (layer F.Fab)
+    (fp_text value 3.9 (at 5.4 0.2) (layer F.Fab)
       (effects (font (size 1 1) (thickness 0.15)))
     )
@@
       (effects (font (size 1 1) (thickness 0.15)))
     )
-    (fp_text value 3.3K (at 5.08 3.81 180) (layer F.Fab)
+    (fp_text value 3.3K (at 4.925 0.15 180) (layer F.Fab)
       (effects (font (size 1 1) (thickness 0.15)))
     )
@@
       (effects (font (size 1 1) (thickness 0.15)))
     )
-    (fp_text value 3.3K (at 5.08 3.81 270) (layer F.Fab)
+    (fp_text value 3.3K (at 4.8 0.2 270) (layer F.Fab)
       (effects (font (size 1 1) (thickness 0.15)))
     )
@@
       (effects (font (size 1 1) (thickness 0.15)))
     )
-    (fp_text value 1N4003 (at 4.37134 -3.55854 90) (layer F.Fab)
+    (fp_text value 1N4003 (at 5.275 -0.225 90) (layer F.Fab)
       (effects (font (size 1 1) (thickness 0.15)))
     )
@@
       (effects (font (size 1 1) (thickness 0.15)))
     )
-    (fp_text value 1N4003 (at 4.37134 -3.55854 90) (layer F.Fab)
+    (fp_text value 1N4003 (at 5 0.05 90) (layer F.Fab)
       (effects (font (size 1 1) (thickness 0.15)))
     )
@@
     (effects (font (size 2 2) (thickness 0.3)))
   )
-  (gr_line (start 63 138) (end 63 38) (angle 90) (layer Eco2.User) (width 0.2))
-  (gr_line (start 193 138) (end 63 138) (angle 90) (layer Eco2.User) (width 0.2))
-  (gr_line (start 193 38) (end 193 138) (angle 90) (layer Eco2.User) (width 0.2))
-  (gr_line (start 63 38) (end 193 38) (angle 90) (layer Eco2.User) (width 0.2))
+  (gr_line (start 63 138) (end 63 38) (angle 90) (layer Edge.Cuts) (width 0.2))
+  (gr_line (start 193 138) (end 63 138) (angle 90) (layer Edge.Cuts) (width 0.2))
+  (gr_line (start 193 38) (end 193 138) (angle 90) (layer Edge.Cuts) (width 0.2))
+  (gr_line (start 63 38) (end 193 38) (angle 90) (layer Edge.Cuts) (width 0.2))
   (gr_line (start 78 123) (end 78 53) (angle 90) (layer Eco1.User) (width 0.2))
   (gr_line (start 178 123) (end 78 123) (angle 90) (layer Eco1.User) (width 0.2))
